File: epilepsyAndBehaviorHat/epilepsyAndBehaviorHat.kicad_pcb (KiCad board)
At the start: 2 copper layers, 100 x 60 mm, 12 parts, among them J1 GPIO, J2 Barrel_Jack_Switch_Pin3Ring, J3 Screw_Terminal_01x02, J4 Screw_Terminal_01x02, Q1 PN2222A

Commit message: Updated PCB
Parts:
- added D2: 1N4001, Diode_THT:D_DO-41_SOD81_P10.16mm_Horizontal, F.Cu at (79.0, 87.0)
- added D3: 1N4001, Diode_THT:D_DO-41_SOD81_P10.16mm_Horizontal, F.Cu at (151.0, 90.1)
- added D4: 1N4001, Diode_THT:D_DO-41_SOD81_P10.16mm_Horizontal, F.Cu at (141.0, 90.1)
- added D5: 1N4001, Diode_THT:D_DO-41_SOD81_P10.16mm_Horizontal, F.Cu at (131.0, 90.1)
- added D6: 1N4001, Diode_THT:D_DO-41_SOD81_P10.16mm_Horizontal, F.Cu at (124.5, 90.1)
- added J10: Screw_Terminal_01x02, TerminalBlock:TerminalBlock_Xinya_XY308-2.54-2P_1x02_P2.54mm_Horizontal, F.Cu at (69.5, 47.1)
- added J11: Screw_Terminal_01x02, TerminalBlock:TerminalBlock_Xinya_XY308-2.54-2P_1x02_P2.54mm_Horizontal, F.Cu at (70.4, 89.5)
- added J12: Screw_Terminal_01x02, TerminalBlock:TerminalBlock_Xinya_XY308-2.54-2P_1x02_P2.54mm_Horizontal, F.Cu at (70.4, 97.2)
- added J13: Conn_01x03_Pin, Connector_PinHeader_2.54mm:PinHeader_1x03_P2.54mm_Vertical, F.Cu at (161.8, 61.8)
- added J14: Screw_Terminal_01x02, TerminalBlock:TerminalBlock_Xinya_XY308-2.54-2P_1x02_P2.54mm_Horizontal, F.Cu at (83.0, 98.6)
- added J15: Screw_Terminal_01x02, TerminalBlock:TerminalBlock_Xinya_XY308-2.54-2P_1x02_P2.54mm_Horizontal, F.Cu at (90.7, 98.6)
- added J16: Screw_Terminal_01x02, TerminalBlock:TerminalBlock_Xinya_XY308-2.54-2P_1x02_P2.54mm_Horizontal, F.Cu at (111.5, 98.6)
- added J5: Screw_Terminal_01x02, TerminalBlock:TerminalBlock_Xinya_XY308-2.54-2P_1x02_P2.54mm_Horizontal, F.Cu at (69.0, 72.0)
- added J6: Screw_Terminal_01x02, TerminalBlock:TerminalBlock_Xinya_XY308-2.54-2P_1x02_P2.54mm_Horizontal, F.Cu at (151.0, 98.0)
- added J7: Screw_Terminal_01x02, TerminalBlock:TerminalBlock_Xinya_XY308-2.54-2P_1x02_P2.54mm_Horizontal, F.Cu at (141.5, 98.0)
- added J8: Screw_Terminal_01x02, TerminalBlock:TerminalBlock_Xinya_XY308-2.54-2P_1x02_P2.54mm_Horizontal, F.Cu at (131.0, 98.0)
- added J9: Screw_Terminal_01x02, TerminalBlock:TerminalBlock_Xinya_XY308-2.54-2P_1x02_P2.54mm_Horizontal, F.Cu at (122.5, 98.0)
- added Q2: PN2222A, Package_TO_SOT_THT:TO-92_Inline, F.Cu at (84.0, 79.7)
- added Q3: PN2222A, Package_TO_SOT_THT:TO-92_Inline, F.Cu at (161.0, 88.2)
- added Q4: PN2222A, Package_TO_SOT_THT:TO-92_Inline, F.Cu at (148.0, 72.0)
- added Q5: PN2222A, Package_TO_SOT_THT:TO-92_Inline, F.Cu at (139.0, 71.7)
- added Q6: PN2222A, Package_TO_SOT_THT:TO-92_Inline, F.Cu at (131.1, 71.7)
- added R4: 220-330, Resistor_THT:R_Axial_DIN0309_L9.0mm_D3.2mm_P12.70mm_Horizontal, F.Cu at (90.0, 81.0)
- added R5: 220-330, Resistor_THT:R_Axial_DIN0309_L9.0mm_D3.2mm_P12.70mm_Horizontal, F.Cu at (161.0, 84.3)
- added R6: 220-330, Resistor_THT:R_Axial_DIN0309_L9.0mm_D3.2mm_P12.70mm_Horizontal, F.Cu at (151.0, 66.7)
- added R7: 220-330, Resistor_THT:R_Axial_DIN0309_L9.0mm_D3.2mm_P12.70mm_Horizontal, F.Cu at (144.0, 66.3)
- added R8: 220-330, Resistor_THT:R_Axial_DIN0309_L9.0mm_D3.2mm_P12.70mm_Horizontal, F.Cu at (137.5, 66.3)
- R3: footprint Resistor_THT:R_Axial_DIN0207_L6.3mm_D2.5mm_P7.62mm_Horizontal -> Resistor_THT:R_Axial_DIN0309_L9.0mm_D3.2mm_P12.70mm_Horizontal
- moved J3 65.0 mm to (69.0, 61.0), turned to -90 degrees
- moved Q1 55.8 mm to (84.0, 67.7), turned to -90 degrees
- moved D1 53.0 mm to (78.9, 74.0)
- moved R3 41.1 mm to (90.0, 69.0)
- moved C2 1.50 mm to (89.0, 62.5)
Connections:
- J3 pad 1: /PWR -> Net-(D1-A)
- J3 pad 2: Net-(D1-A) -> /PWR
- R3 pad 1: /GPIO26 -> Net-(Q1-B)
- R3 pad 2: Net-(Q1-B) -> /GPIO17
Routing:
- net /PWR: track 10.0 -> 205.2 mm, vias 0 -> 3
- net GND: track 106.4 -> 248.3 mm
- net /GPIO25: track 0.00 -> 94.3 mm
- net /GPIO24: track 0.00 -> 88.5 mm
- net /GPIO23: track 0.00 -> 83.0 mm
- net /GPIO22: track 0.00 -> 82.0 mm
- net /GPIO10/SPI0.MOSI: track 0.00 -> 78.6 mm, vias 0 -> 1
- net /GPIO27: track 0.00 -> 40.9 mm
- net unconnected-(J14-Pin_2-Pad2): track 0.00 -> 37.7 mm
- net unconnected-(J15-Pin_1-Pad1): track 0.00 -> 33.3 mm
- net unconnected-(J15-Pin_2-Pad2): track 0.00 -> 31.5 mm
- net Net-(D6-A): track 0.00 -> 30.3 mm
- net Net-(D5-A): track 0.00 -> 29.5 mm
- net /GPIO26: track 0.00 -> 28.6 mm, vias 0 -> 1
- net Net-(D4-A): track 0.00 -> 28.6 mm
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Other:
- board text added: "GPIO23 GPIO22 GPIO24 GPIO25"
- board text added: "MOTOR B (GPIO 27)"
- board text added: "MOTOR C (GPIO 5)"
- board text added: "MOTOR D (GPIO 6)"
- board text added: "MOTOR E (GPIO 16)"
- board text added: "MOTOR F (GPIO 26)"
- board text added: "Motor A (GPIO 17)"
- board text added: "PWR GND"
