File: epilepsyAndBehaviorHat/epilepsyAndBehaviorHat.kicad_sch (KiCad schematic)
At the start: 13 parts, among them J1 GPIO, J2 Barrel_Jack_Switch_Pin3Ring, J3 Screw_Terminal_01x02, J4 Screw_Terminal_01x02, Q1 PN2222A, U1 CAT24C256

Commit message: Updated PCB
Parts:
- added D2, D3, D4, D5, D6: 1N4001, Diode_THT:D_DO-41_SOD81_P10.16mm_Horizontal, symbol Diode:1N4001
- added J10, J11, J12, J14, J15, J16, J5, J6, J7, J8, J9: Screw_Terminal_01x02, TerminalBlock:TerminalBlock_Xinya_XY308-2.54-2P_1x02_P2.54mm_Horizontal, symbol Connector:Screw_Terminal_01x02
- added J13: Conn_01x03_Pin, Connector_PinHeader_2.54mm:PinHeader_1x03_P2.54mm_Vertical, symbol Connector:Conn_01x03_Pin
- added Q2, Q3, Q4, Q5, Q6: PN2222A, Package_TO_SOT_THT:TO-92_Inline, symbol Transistor_BJT:PN2222A
- added R4, R5, R6, R7, R8: 220-330, Resistor_THT:R_Axial_DIN0309_L9.0mm_D3.2mm_P12.70mm_Horizontal, symbol Device:R_US
- C2: footprint Capacitor_THT:C_Axial_L12.0mm_D10.5mm_P15.00mm_Horizontal -> Capacitor_THT:C_Axial_L5.1mm_D3.1mm_P10.00mm_Horizontal
- R3: footprint Resistor_THT:R_Axial_DIN0207_L6.3mm_D2.5mm_P7.62mm_Horizontal -> Resistor_THT:R_Axial_DIN0309_L9.0mm_D3.2mm_P12.70mm_Horizontal
Connections:
- net GND: now also J10.2 (Pin_2), Q2.1 (E), Q3.1 (E), Q4.1 (E), Q5.1 (E), Q6.1 (E)
- net GPIO10/SPI0.MOSI: now also J14.1 (Pin_1)
- net GPIO16: now also R6.2
- net GPIO17: now also R3.2
- net GPIO19/PCM.FS: now also J13.3 (Pin_3)
- net GPIO20/PCM.DIN: now also J13.2 (Pin_2)
- net GPIO21/PCM.DOUT: now also J13.1 (Pin_1)
- net GPIO22: now also J11.2 (Pin_2)
- net GPIO23: now also J11.1 (Pin_1)
- net GPIO24: now also J12.1 (Pin_1)
- net GPIO25: now also J12.2 (Pin_2)
- net GPIO26: now also R5.2; no longer R3.1
- net GPIO27: now also R4.2
- net GPIO5: now also R8.2
- net GPIO6: now also R7.2
- net PWR: now also J3.2 (Pin_2), D2.1 (K), D3.1 (K), D4.1 (K), D5.1 (K), D6.1 (K), J10.1 (Pin_1), J5.2 (Pin_2), J6.1 (Pin_1), J7.1 (Pin_1), J8.1 (Pin_1), J9.1 (Pin_1); no longer J3.1 (Pin_1)
- net at D1.2 (A), Q1.3 (C): now also J3.1 (Pin_1); no longer J3.2 (Pin_2)
- net at Q1.2 (B): now also R3.1; no longer R3.2
- new net: D4.2 (A), J7.2 (Pin_2), Q4.3 (C)
- new net: D6.2 (A), J9.2 (Pin_2), Q6.3 (C)
- new net: D3.2 (A), J6.2 (Pin_2), Q3.3 (C)
- new net: Q4.2 (B), R6.1
- new net: Q6.2 (B), R8.1
- new net: Q5.2 (B), R7.1
- new net: D5.2 (A), J8.2 (Pin_2), Q5.3 (C)
- new net: Q3.2 (B), R5.1
- new net: Q2.2 (B), R4.1
- new net: D2.2 (A), J5.1 (Pin_1), Q2.3 (C)
Other:
- moved on the sheet: D1, J3, Q1, R3
